File: PCB/HexaDecipad-V3/HexaDecipad-V3.kicad_pcb (KiCad board)
At the start: 2 copper layers, 85 x 90 mm, 25 parts, among them SW1 RotaryEncoder_Switch, SW10 SW_Push_45deg, SW11 SW_Push_45deg, SW12 SW_Push_45deg, SW2 RotaryEncoder_Switch, SW3 SW_Push_45deg, SW4 SW_Push_45deg, SW5 SW_Push_45deg, SW6 SW_Push_45deg, SW7 SW_Push_45deg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

Commit message: pushing stuff
Parts:
- D10, D11, D12, D3, D4, D5, D6, D7, D8, D9, SW10, SW11, SW12, SW3, SW4, SW5, SW6, SW7, SW8, SW9: moved to B.Cu
- moved D7 226.6 mm to (269.4, 125.0), turned to 180 degrees
- moved D6 221.5 mm to (269.4, 106.0), turned to 180 degrees
- moved D2 211.0 mm to (261.4, 81.8)
- moved D12 209.5 mm to (250.4, 144.0), turned to 180 degrees
- moved D8 207.7 mm to (250.4, 125.0), turned to 180 degrees
- moved D5 204.7 mm to (250.4, 106.0), turned to 180 degrees
- moved D11 193.8 mm to (231.4, 144.0), turned to 180 degrees
- moved D9 188.8 mm to (231.4, 125.0), turned to 180 degrees
- moved D4 188.3 mm to (231.4, 106.0), turned to 180 degrees
- moved D1 173.3 mm to (220.6, 82.0), turned to 180 degrees
- moved D3 172.5 mm to (212.4, 106.0), turned to 180 degrees
- moved D10 170.0 mm to (212.4, 125.0), turned to 180 degrees
- moved SW1 6.46 mm to (209.5, 89.5)
- moved SW2 6.46 mm to (257.5, 89.5)
- turned SW10 to 180 degrees
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Routing:
- net /Row 2: track 0.00 -> 119.8 mm
- net /Row 1: track 0.00 -> 105.3 mm
- net /Row 3: track 0.00 -> 62.9 mm
- net /Column 2: track 0.00 -> 45.7 mm
- net /Column 3: track 0.00 -> 43.4 mm
- net /Column 1: track 0.00 -> 29.3 mm, vias 0 -> 1
- net /Column 4: track 0.00 -> 29.0 mm
- net Net-(D1-A): track 0.00 -> 18.5 mm
- net Net-(D2-A): track 0.00 -> 13.9 mm
- net Net-(D12-A): track 0.00 -> 6.68 mm
- net Net-(D11-A): track 0.00 -> 6.65 mm
- net Net-(D7-A): track 0.00 -> 6.65 mm
- net Net-(D8-A): track 0.00 -> 6.63 mm
- net Net-(D9-A): track 0.00 -> 6.60 mm
- net Net-(D6-A): track 0.00 -> 6.60 mm
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